File: v1/v1.kicad_sch (KiCad schematic)
At the start: 7 parts, among them J1 Conn_02x22_Top_Bottom, U1 ESP32-S3-DevKitC, U2 DM-OLED096-636

Commit message: code, new pcb and bom
Parts:
- removed J1: Conn_02x22_Top_Bottom, Connector_PinHeader_2.54mm:PinHeader_2x22_P2.54mm_Vertical, symbol Connector_Generic:Conn_02x22_Top_Bottom
- removed U2: DM-OLED096-636, Library:MODULE_DM-OLED096-636, symbol DM-OLED096-636:DM-OLED096-636
- added DS1: OLED_128X64_1.3_I2C, LCD_OLED_128X64_1.3_I2C:LCD_OLED_128X64_1.3_I2C, symbol OLED_128X64_1.3_I2C:OLED_128X64_1.3_I2C
- added L1: (no value), Connector_PinHeader_2.54mm:PinHeader_1x08_P2.54mm_Vertical, symbol New_Library:LCD_1
- added T1: (no value), Connector_PinHeader_2.54mm:PinHeader_1x03_P2.54mm_Vertical, symbol New_Library:_TTP223
Connections:
- net at U1.1 (3V3), U1.2 (3V3): now also DS1.1 (VDD), L1.2 (VCC), L1.8 (BL), T1.3 (VCC)
- net at U1.10 (GPIO17/ADC2_CH6): now also L1.4 (SDA)
- net at U1.11 (GPIO18/ADC2_CH7): now also L1.3 (SCL)
- net at U1.22 (GND), U1.23 (GND), U1.24 (GND)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: now also DS1.2 (GND), L1.1 (GND), T1.1 (GND)
- net at U1.40 (GPIO2/ADC1_CH1): now also L1.6 (DC)
- net at U1.4 (GPIO4/ADC1_CH3): now also L1.5 (RES)
- net at U1.5 (GPIO5/ADC1_CH4): now also L1.7 (CS)
- net at U1.7 (GPIO7/ADC1_CH6): now also DS1.3 (SCK)
- net at U1.8 (GPIO15/ADC2_CH4/32K_P): now also T1.2 (IO)
- net at U1.9 (GPIO16/ADC2_CH5/32K_N): now also DS1.4 (SDA)

Commit message: new PCB schematic, readme, BOM
Parts:
- removed U1: ESP32-S3-DevKitC, PCM_Espressif:ESP32-S3-DevKitC, symbol PCM_Espressif:ESP32-S3-DevKitC
- added C1, C2: GRM188R60J106KE47D, footprints:CAP_GRM188_1608_MUR, symbol 2026-04-10_19-44-45:GRM188R60J106KE47D
- added J1: CX90BW1-24P1, footprints:HIROSE_CX90BW1-24P1, symbol CX90BW1-24P1:CX90BW1-24P1
- added R1, R2: RC0402FR-075K1L, footprints:RC0402N_YAG, symbol 2026-04-10_19-50-19:RC0402FR-075K1L
- added R3, R4: 10k, Resistor_THT:R_Axial_DIN0207_L6.3mm_D2.5mm_P10.16mm_Horizontal, symbol SL_Resistors:10k
- added SW1, SW2: SKRPABE010, SW4_SKRPABE010_ALPS, symbol 2026-04-10_19-33-01:SKRPABE010
- added U1: TLV1117-33IDCYR, footprints:DCY0004A_L, symbol 2026-04-10_19-32-37:TLV1117-33IDCYR
- added U2: ESP32-S3-WROOM-1, PCM_Espressif:ESP32-S3-WROOM-1, symbol PCM_Espressif:ESP32-S3-WROOM-1
Connections:
- net 3V3: now reaches DS1.1 (VDD), L1.2 (VCC), L1.8 (BL), T1.3 (VCC)
- net 3V3: now also C1.2, C2.2, U2.2 (3V3)
- net GND_A: now reaches DS1.2 (GND), L1.1 (GND), T1.1 (GND)
- net GND_A: now also J1.A1 (GND_A), J1.A12 (GND_A), J1.B1 (GND_B), J1.B12 (GND_B), J1.SH1 (SHIELD), J1.SH2 (SHIELD), J1.SH3 (SHIELD), J1.SH4 (SHIELD), R1.2, R2.1, SW1.3, SW1.4, SW2.3, SW2.4, U1.1 (GND), U2.1 (GND), U2.40 (GND), U2.41 (GND)
- net GPIO7: now reaches DS1.3 (SCK)
- net GPIO7: now also U2.7 (GPIO7/TOUCH7/ADC1_CH6)
- net GPIO16: now reaches DS1.4 (SDA)
- net GPIO16: now also U2.9 (GPIO16/U0CTS/ADC2_CH5/XTAL_32K_N)
- net GPIO17: now reaches L1.4 (SDA)
- net GPIO17: now also U2.10 (GPIO17/U1TXD/ADC2_CH6)
- net GPIO18: now reaches L1.3 (SCL)
- net GPIO18: now also U2.11 (GPIO18/U1RXD/ADC2_CH7/CLK_OUT3)
- net GPIO4: now reaches L1.5 (RES)
- net GPIO4: now also U2.4 (GPIO4/TOUCH4/ADC1_CH3)
- net GPIO2: now reaches L1.6 (DC)
- net GPIO2: now also U2.38 (GPIO2/TOUCH2/ADC1_CH1)
- net GPIO5: now reaches L1.7 (CS)
- net GPIO5: now also U2.5 (GPIO5/TOUCH5/ADC1_CH4)
- net GPIO15: now reaches T1.2 (IO)
- net GPIO15: now also U2.8 (GPIO15/U0RTS/ADC2_CH4/XTAL_32K_P)
- new net: C1.1, U1.2 (OUTPUT)
- new net: C2.1, U1.4 (OUTPUT)
- new net: R4.1, U2.27 (GPIO0/BOOT)
- new net: R3.2, U2.3 (EN)
- new net: J1.B5 (CC2), R2.2
- new net: J1.A5 (CC1), R1.1
- new net BOOT: R4.2, SW1.1, SW1.2
- new net D+: J1.A6 (D1+), U2.14 (GPIO20/U1CTS/ADC2_CH9/CLK_OUT1/USB_D+)
- new net D-: J1.A7 (D1-), U2.13 (GPIO19/U1RTS/ADC2_CH8/CLK_OUT2/USB_D-)
- new net EN: R3.1, SW2.1, SW2.2
- new net VBUS_A: J1.A4 (VBUS_A), J1.A9 (VBUS_A), U1.3 (IN)
- new net VBUS_B: J1.B4 (VBUS_B), J1.B9 (VBUS_B)
